File: carte_mere.kicad_pcb (KiCad board)
At the start: 4 copper layers, 56.8 x 142 mm, 266 parts, among them J1 Conn_01x02_Pin, J10 Conn_01x02_Pin, J11 Conn_01x02_Pin, J12 Conn_01x02_Pin, J13 Conn_01x03_Pin, J14 Conn_01x02, J15 Conn_01x04, J16 Conn_01x03_Pin, J17 Conn_01x05_Pin, J18 Conn_01x02, J19 Conn_01x02, J2 Conn_01x03_Pin, J20 Conn_01x04, J21 Conn_01x04, J22 Conn_01x04, J23 Conn_01x03, J24 Conn_01x02, J25 Conn_01x03_Pin, J26 Conn_01x03_Pin, J27 Conn_01x03_Pin, J28 Conn_01x03_Pin, J29 Conn_01x03_Pin, J3 Conn_01x03_Pin, J30 Conn_01x03_Pin, J31 Conn_01x03_Pin, J32 Conn_01x03_Pin, J33 Conn_01x03_Pin, J34 Conn_01x03_Pin, J35 Conn_01x03_Pin, J36 Conn_01x03_Pin, J37 Conn_01x03_Pin, J38 Conn_01x03_Pin, J39 Conn_01x05_Pin, J4 Conn_01x03_Pin, J40 Conn_01x05_Pin, J41 Conn_01x06_Pin, J42 Conn_01x06_Pin, J43 Conn_01x02_Pin, J5 Conn_01x03_Pin, J6 Conn_01x03_Pin, J7 Conn_01x03_Pin, J8 Conn_01x03_Pin, J9 Conn_01x03_Pin, Q19 2N7002, Q20 2N7002, Q21 2N7002, Q22 2N7002, Q23 2N7002, Q24 2N7002, Q25 2N7002, Q26 2N7002, Q27 2N7002, Q28 2N7002, Q29 2N7002, Q30 2N7002, Q31 2N7002, Q32 2N7002, Q33 2N7002, Q34 2N7002, Q35 2N7002, Q37 2N7002, Q38 2N7002, Q39 2N7002, Q40 2N7002, U1 SN65HVD230, U10 SN74LV1T34DCK, U11 SN74LV1T34DCK, U12 SN74LV1T34DCK, U13 SN74LV1T34DCK, U2 SN74LVC1T45DBV, U3 SN74LV1T34DCK, U4 SN74LV1T34DCK, U5 TPS54302, U6 TPS54302, U7 SN74LV1T34DCK, U8 SN74LV1T34DCK, U9 SN74LV1T34DCK

Commit message: clean
Parts:
- removed D2: LED, LED_SMD:LED_0402_1005Metric
- removed R33: 1k, Resistor_SMD:R_0402_1005Metric
Routing:
- net AX_DATA: track 97.4 -> 94.9 mm
- net 3.3V: track 125.0 -> 123.3 mm, vias 26 -> 25
- net Net-(D2-K): track 1.35 -> 0.00 mm
- net AX_DIR: track 106.3 -> 105.7 mm

Commit message: update
Parts:
- Q35: footprint Package_TO_SOT_SMD:TSOT-23 -> Package_TO_SOT_SMD:SOT-23
